File: hub75-adapter.kicad_sch (KiCad schematic)
At the start: 9 parts, among them J1 PI, J2 5V_IN, J3 HUB75, J4 5V_OUT_MATRIX

Commit message: rev2 w/ oe resistor
Parts:
- added R1: 10k, Resistor_THT:R_Axial_DIN0207_L6.3mm_D2.5mm_P7.62mm_Horizontal, symbol Device:R
- JP1, JP2: footprint Jumper:SolderJumper-3_P1.3mm_Bridged12_Pad1.0x1.5mm -> Jumper:SolderJumper-3_P1.3mm_Open_Pad1.0x1.5mm; symbol Jumper:SolderJumper_3_Bridged12 -> Jumper:SolderJumper_3_Open
Connections:
- net ~{OE}: now also R1.1
- net +3V3: now reaches J1.1 (3V3), J1.17 (3V3)
- net +3V3: now also R1.2
- no-connect marks 15 -> 14
